Commit message: add working moveit config, see install.sh for notes

File: cora_description/urdf/cora.urdf (robot description, URDF)
Before this commit: robot cora, 13 links, 12 joints
Links:
- link baselink: geometry collision mesh filename=package://cora_description/meshes/cora/merged/baselink_coll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; visual mesh filename=package://cora_description/meshes/cora/merged/baselink_visu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
- link endeffector: geometry collision mesh filename=package://cora_description/meshes/cora/merged/endeffector_c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; visual mesh filename=package://cora_description/meshes/cora/merged/endeffector_v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
- link gripper_body: geometry collision mesh filename=package://cora_description/meshes/cora/merged/gripper_body_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; visual mesh filename=package://cora_description/meshes/cora/merged/gripper_body_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
- link gripper_fingers: geometry collision mesh filename=package://cora_description/meshes/cora/merged/gripper_finge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; visual mesh filename=package://cora_description/meshes/cora/merged/gripper_finge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
- link gripper_fingers_2: geometry collision mesh filename=package://cora_description/meshes/cora/merged/gripper_finge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; visual mesh filename=package://cora_description/meshes/cora/merged/gripper_finge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
- link l1: geometry collision mesh filename=package://cora_description/meshes/cora/merged/l1_collision.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; visual mesh filename=package://cora_description/meshes/cora/merged/l1_visual.stl
- link l2: geometry collision mesh filename=package://cora_description/meshes/cora/merged/l2_collision.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; visual mesh filename=package://cora_description/meshes/cora/merged/l2_visual.stl
- link l3: geometry collision mesh filename=package://cora_description/meshes/cora/merged/l3_collision.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; visual mesh filename=package://cora_description/meshes/cora/merged/l3_visual.stl
- link l4: geometry collision mesh filename=package://cora_description/meshes/cora/merged/l4_collision.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; visual mesh filename=package://cora_description/meshes/cora/merged/l4_visual.stl
- link l5: geometry collision mesh filename=package://cora_description/meshes/cora/merged/l5_collision.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; visual mesh filename=package://cora_description/meshes/cora/merged/l5_visual.stl

Commit message: fixed parallel gripper command controller

File: cora_description/urdf/cora.urdf (robot description, URDF)
Before this commit: robot cora, 13 links, 12 joints
Joints:
- joint Finger1: limit lower=2.45463e-16 upper=0.0385 effort=10 velocity=10 -> lower=0.0 upper=0.0385 effort=10 velocity=10
- joint Finger2: limit lower=-1.60028e-15 upper=0.0385 effort=10 velocity=10 -> lower=0.0 upper=0.0385 effort=10 velocity=10

Commit message: abstracted gripper away from main urdf. pass gripper package name as launch argument to move.launch and it will load xacro and urdf files accordingly

File: cora_description/urdf/cora.urdf (robot description, URDF)
Before this commit: robot cora, 13 links, 12 joints
Links:
- removed link Camera
- removed link Gripper
- removed link gripper_body
- removed link gripper_fingers
- removed link gripper_fingers_2
Joints:
- removed joint Camera_frame
- removed joint Finger1
- removed joint Finger2
- removed joint GripperFix
- removed joint Gripper_frame

File: cora_moveit_config/config/cora.ros2_control.xacro (robot description, xacro)
@@ -1,10 +1,17 @@
 <?xml version="1.0"?>
 <robot xmlns:xacro="http://www.ros.org/wiki/xacro">
-    <xacro:macro name="cora_ros2_control" params="name initial_positions_file">
+    <xacro:macro name="cora_ros2_control" params="name initial_positions_file hardware_type">
         <xacro:property name="initial_positions" value="${xacro.load_yaml(initial_positions_file)['initial_positions']}"/>
         <ros2_control name="${name}" type="system">
             <hardware>
-                <!-- By default, set up controllers for simulation. This won't work on real hardware -->
-                <plugin>mock_components/GenericSystem</plugin>
+              <!-- By default, set up controllers for fake system-->
+              <xacro:if value="${hardware_type == 'Fake'}">
+                <plugin>mock_components/GenericSystem</plugin> <!-- Mock Components -->
+              </xacro:if>
+              <!-- Real Hardware Components -->
+              <xacro:if value="${hardware_type == 'Real'}">
+                <plugin>odrive_ros2_control_plugin/odriveHardwareInterface</plugin>
+                <param name="can">can0</param>
+              </xacro:if>
             </hardware>
             <joint name="J1">
@@ -15,4 +22,5 @@
                 </state_interface>
                 <state_interface name="velocity"/>
+                <param name="node_id">0</param>
             </joint>
             <joint name="J2">
@@ -23,4 +31,5 @@
                 </state_interface>
                 <state_interface name="velocity"/>
+                <param name="node_id">1</param>
             </joint>
             <joint name="J3">
@@ -31,4 +40,5 @@
                 </state_interface>
                 <state_interface name="velocity"/>
+                <param name="node_id">2</param>
             </joint>
             <joint name="J4">
@@ -39,4 +49,5 @@
                 </state_interface>
                 <state_interface name="velocity"/>
+                <param name="node_id">3</param>
             </joint>
             <joint name="J5">
@@ -47,4 +58,5 @@
                 </state_interface>
                 <state_interface name="velocity"/>
+                <param name="node_id">4</param>
             </joint>
             <joint name="J6">
@@ -55,12 +67,5 @@
                 </state_interface>
                 <state_interface name="velocity"/>
-            </joint>
-            <joint name="Finger1">
-                <command_interface name="position"/>
-                <command_interface name="velocity"/>
-                <state_interface name="position">
-                  <param name="initial_value">${initial_positions['Finger1']}</param>
-                </state_interface>
-                <state_interface name="velocity"/>
+                <param name="node_id">5</param>
             </joint>
         </ros2_control>

File: cora_moveit_config/config/cora.urdf.xacro (robot description, xacro)
@@ -1,9 +1,41 @@
 <?xml version="1.0"?>
 <robot xmlns:xacro="http://www.ros.org/wiki/xacro" name="cora">
-    <xacro:arg name="initial_positions_file" default="initial_positions.yaml" />
-    <!-- Import cora urdf file -->
-    <xacro:include filename="$(find cora_description)/urdf/cora.urdf" />
-    <!-- Import control_xacro -->
-    <xacro:include filename="cora.ros2_control.xacro" />
-    <xacro:cora_ros2_control name="FakeSystem" initial_positions_file="$(arg initial_positions_file)"/>
+    <!-- ================= -->
+    <!-- Declare arguments -->
+    <!-- ================= -->
+    <xacro:arg name="hardware_type" default="Fake"/>
+    <xacro:arg name="gripper_package" default="None"/>
+    <xacro:arg name="initial_positions_file" default="initial_positions.yaml"/>
+    <!-- ================= -->
+    <!-- Base robot        -->
+    <!-- ================= -->
+    <xacro:include filename="$(find cora_description)/urdf/cora.urdf"/>
+    <!-- ================= -->
+    <!-- ros2_control      -->
+    <!-- ================= -->
+    <xacro:include filename="cora.ros2_control.xacro"/>
+    <xacro:cora_ros2_control
+        name="CoraSystem"
+        hardware_type="$(arg hardware_type)"
+        initial_positions_file="$(arg initial_positions_file)"/>
+    <!-- ================= -->
+    <!-- Optional gripper  -->
+    <!-- ================= -->
+    <!-- Store gripper package -->
+    <xacro:property
+        name="gripper_package_name"
+        value="$(arg gripper_package)"/>
+    <!-- Store gripper package path -->
+    <xacro:property
+        name="gripper_package_path"
+        value="$(find ${gripper_package_name})"/>
+    <!-- Only load gripper if one is provided -->
+    <xacro:if value="${gripper_package_name != 'None'}">
+        <!-- Load gripper macros -->
+        <xacro:include filename="${gripper_package_path}/urdf/cora_gripper.urdf.xacro"/>
+        <!-- Instantiate gripper -->
+        <xacro:cora_gripper_xacro
+            hardware_type="$(arg hardware_type)"
+            initial_positions_file="$(arg initial_positions_file)"/>
+    </xacro:if>
 </robot>
