Commit message: added real geometry for 3 joints in the test description

File: odrive_ros2_control/config/test_joint.urdf (robot description, URDF)
Before this commit: robot test_joint_robot, 3 links, 2 joints
Links:
- removed link arm_link_1
- removed link arm_link_2
- link base_link: mass None -> 0
Joints:
- removed joint test_joint_1
- removed joint test_joint_2
